Commit message: Updated URDF.

File: lynxmotion_al5d_support/urdf/al5d.urdf (robot description, URDF)
Before this commit: robot lynxmotion_al5d, 6 links, 5 joints
Links:
- removed link gripper
- removed link link_1
- removed link link_2
- removed link link_3
- removed link link_4
- added link finger_base; collision box size=0.0385 0.065 0.0195; visual box size=0.0385 0.065 0.0195
- added link forearm; collision box size=0.078 0.070 0.034; collision box size=0.181 0.054 0.026
- added link hand; collision box size=0.063 0.078 0.024; visual box size=0.063 0.078 0.024
- added link left_finger; collision box size=0.0285 0.0135 0.019; visual box size=0.0285 0.0135 0.019
- added link right_finger; collision box size=0.0285 0.0135 0.019; visual box size=0.0285 0.0135 0.019
- added link shoulder_servo_link; collision box size=0.061 0.082 0.037; visual box size=0.061 0.082 0.037
- added link upper_arm; collision box size=0.024 0.078 0.18; visual box size=0.024 0.078 0.18
- link base_link: geometry collision cylinder length=0.056 radius=0.0475; visual cylinder length=0.056 radius=0.0475
Joints:
- removed joint end_effector
- removed joint joint_1
- removed joint joint_2
- removed joint joint_3
- removed joint joint_4
- added joint base_joint: type revolute, parent base_link, child shoulder_servo_link, origin xyz=0 0 0.0465 rpy=0 0 0, axis 0 0 1, limit lower=-1.57 upper=1.57 effort=10 velocity=3
- added joint elbow: type revolute, parent upper_arm, child forearm, origin xyz=0 0 0.167 rpy=0 0 0, axis 0 1 0, limit lower=-1.57 upper=1.57 effort=10 velocity=3
- added joint left_gripper: type prismatic, parent finger_base, child left_finger, origin xyz=0.0335 0.02375 0 rpy=0 0 0, axis 0 1 0, limit lower=-0.017 upper=0 effort=10 velocity=3
- added joint right_gripper: type prismatic, parent finger_base, child right_finger, origin xyz=0.0335 -0.02375 0 rpy=0 0 0, axis 0 1 0, limit lower=-0.017 upper=0 effort=10 velocity=3, mimic joint=left_gripper multiplier=-1
- added joint shoulder_joint: type revolute, parent shoulder_servo_link, child upper_arm, axis 0 1 0, limit lower=-1.553 upper=1.553 effort=0 velocity=3
- added joint wrist: type revolute, parent forearm, child hand, origin xyz=0.189 0 0, axis 0 1 0, limit lower=-1.57 upper=1.57 effort=10 velocity=3
- added joint wrist_rotate: type revolute, parent hand, child finger_base, origin xyz=0.07 0 0, axis 1 0 0, limit lower=-1.57 upper=1.57 effort=10 velocity=3
