Commit message: Fixed joint name in URDF.

File: lynxmotion_al5d_support/urdf/al5d.xacro (robot description, xacro)
@@ -1,5 +1,8 @@
 <?xml version="1.0" ?>
 <robot name="lynxmotion_al5d" xmlns:xacro="http://ros.org/wiki/xacro">
+  <link name="base_link"/>
   <xacro:include filename="$(find lynxmotion_al5d_support)/urdf/al5d_macro.xacro"/>
-  <xacro:lynxmotion_al5d prefix=""/>
+  <lynxmotion_al5d prefix="al5d_" parent_link="base_link">
+    <origin xyz="0 0 0"/>
+  </lynxmotion_al5d>
 </robot>

File: lynxmotion_al5d_support/urdf/al5d_macro.xacro (robot description, xacro)
@@ -1,4 +1,5 @@
 <?xml version="1.0"?>
 <robot xmlns:xacro="http://ros.org/wiki/xacro">
+  <xacro:property name="M_PI" value="3.14159"/>
   <property name="base_height" value="0.043" />
   <property name="base_radius" value="0.048" />
@@ -10,5 +11,11 @@
   <property name="link4_length" value="0.032" />
   <property name="gripper_offset" value="0.016" />
-  <xacro:macro name="lynxmotion_al5d" params="prefix">
+  <xacro:macro name="lynxmotion_al5d" params="prefix parent_link *origin">
+    <!-- attach -->
+    <joint name="arm_base_joint" type="fixed">
+      <insert_block name="origin" />
+      <parent link="${parent_link}"/>
+      <child link="${prefix}base_link" />
+    </joint>
     <!-- links -->
     <link name="${prefix}base_link">
@@ -120,5 +127,5 @@
       <child link="${prefix}link_1"/>
       <axis xyz="0 0 -1"/>
-      <limit lower="-1.57079632679" upper="1.57079632679" effort="0" velocity="3.67"/>
+      <limit lower="-${M_PI/2}" upper="${M_PI/2}" effort="0" velocity="3.67"/>
     </joint>
     <joint name="${prefix}joint_2" type="revolute">
@@ -127,12 +134,12 @@
       <child link="${prefix}link_2"/>
       <axis xyz="0 -1 0"/>
-      <limit lower="-1.57079632679" upper="1.57079632679" effort="0" velocity="3.32"/>
+      <limit lower="-${M_PI/2}" upper="${M_PI/2}" effort="0" velocity="3.32"/>
     </joint>
     <joint name="${prefix}joint_3" type="revolute">
-      <origin xyz="0 0 ${link2_length}" rpy="0 1.57079632679 0" />
+      <origin xyz="0 0 ${link2_length}" rpy="0 ${M_PI/2} 0" />
       <parent link="${prefix}link_2"/>
       <child link="${prefix}link_3"/>
       <axis xyz="0 1 0"/>
-      <limit lower="-1.57079632679" upper="1.57079632679" effort="0" velocity="3.67"/>
+      <limit lower="-${M_PI/2}" upper="${M_PI/2}" effort="0" velocity="3.67"/>
     </joint>
     <joint name="${prefix}joint_4" type="revolute">
@@ -141,12 +148,12 @@
       <child link="${prefix}link_4"/>
       <axis xyz="0 -1 0"/>
-      <limit lower="-1.57079632679" upper="1.57079632679" effort="0" velocity="6.98"/>
+      <limit lower="-${M_PI/2}" upper="${M_PI/2}" effort="0" velocity="6.98"/>
     </joint>
-    <joint name="${prefix}end_effector" type="revolute">
+    <joint name="${prefix}gripper" type="revolute">
       <origin xyz="0 0 ${link4_length + gripper_offset}" rpy="0 0 0"/>
       <parent link="${prefix}link_4"/>
       <child link="${prefix}gripper"/>
       <axis xyz="-1 0 0"/>
-      <limit lower="-1.57079632679" upper="1.57079632679" effort="0" velocity="6.98"/>
+      <limit lower="-${M_PI/2}" upper="${M_PI/2}" effort="0" velocity="6.98"/>
     </joint>
   </xacro:macro>
