Commit message: Updated URDF for new zero displacement.

File: lynxmotion_al5d_support/urdf/al5d_macro.xacro (robot description, xacro)
@@ -55,7 +55,7 @@
     <link name="${prefix}link_2">
       <visual>
-        <origin xyz="0 0 ${base_height + link1_height + link2_offset}" rpy="0 0 0"/>
+        <origin xyz="${link2_length/2} 0 0" rpy="0 0 0"/>
         <geometry>
-          <box size="0.02 .02 ${link2_length-0.02}"/>
+          <box size="${link2_length-0.02} 0.02 .02"/>
         </geometry>
         <material name="silver">
@@ -64,7 +64,7 @@
       </visual>
       <collision>
-        <origin xyz="0 0 ${base_height + link1_height + link2_offset}" rpy="0 0 0"/>
+        <origin xyz="${link2_length/2} 0 0" rpy="0 0 0"/>
         <geometry>
-          <box size="0.02 .02 ${link2_length}"/>
+          <box size="${link2_length-0.02} 0.02 .02"/>
         </geometry>
       </collision>
@@ -72,7 +72,7 @@
     <link name="${prefix}link_3">
       <visual>
-        <origin xyz="0 0 ${link3_length/2}" rpy="0 0 0"/>
+        <origin xyz="${link3_length/2} 0 0" rpy="0 0 0"/>
         <geometry>
-          <box size="0.02 0.02 ${link3_length-0.02}"/>
+          <box size="${link3_length-0.02} 0.02 0.02"/>
         </geometry>
         <material name="silver">
@@ -81,7 +81,7 @@
       </visual>
       <collision>
-        <origin xyz="0 0 ${link3_length/2}" rpy="0 0 0"/>
+        <origin xyz="${link3_length/2} 0 0" rpy="0 0 0"/>
         <geometry>
-          <box size="0.02 0.02 ${link3_length}"/>
+          <box size="${link3_length} 0.02 0.02"/>
         </geometry>
       </collision>
@@ -89,7 +89,7 @@
     <link name="${prefix}link_4">
       <visual>
-        <origin xyz="0 0 ${link4_length/2}" rpy="0 0 0"/>
+        <origin xyz="${link4_length/2} 0 0" rpy="0 0 0"/>
         <geometry>
-          <box size="0.02 0.02 ${link4_length}"/>>
+          <box size="${link4_length} 0.02 0.02"/>
         </geometry>
         <material name="black">
@@ -98,7 +98,7 @@
       </visual>
       <collision>
-        <origin xyz="0 0 ${link4_length/2}" rpy="0 0 0"/>
+        <origin xyz="${link4_length/2} 0 0" rpy="0 0 0"/>
         <geometry>
-          <box size="0.02 0.02 ${link4_length}"/>
+          <box size="${link4_length} 0.02 0.02"/>
         </geometry>
       </collision>
@@ -106,5 +106,5 @@
     <link name="${prefix}gripper">
       <visual>
-        <origin xyz="0 0 0.025" rpy="0 0 0"/>
+        <origin xyz="0 0 0" rpy="0 0 0"/>
         <geometry>
           <box size="0.05 0.05 0.05"/>
@@ -123,36 +123,36 @@
     <!-- joints -->
     <joint name="${prefix}joint_1" type="revolute">
-      <origin xyz="0 0 ${base_height + link1_height/2}" rpy="0 0 0"/>
+      <origin xyz="0 0 ${base_height + link1_height}" rpy="0 0 0"/>
       <parent link="${prefix}base_link"/>
       <child link="${prefix}link_1"/>
-      <axis xyz="0 0 -1"/>
+      <axis xyz="0 0 1"/>
       <limit lower="-${M_PI/2}" upper="${M_PI/2}" effort="0" velocity="3.67"/>
     </joint>
     <joint name="${prefix}joint_2" type="revolute">
-      <origin xyz="0 0 ${link2_offset}" rpy="0 0 0"/>
+      <origin xyz="0 0 ${link2_offset}" rpy="${M_PI/2} 0 0"/>
       <parent link="${prefix}link_1"/>
       <child link="${prefix}link_2"/>
-      <axis xyz="0 -1 0"/>
+      <axis xyz="0 0 1"/>
       <limit lower="-${M_PI/2}" upper="${M_PI/2}" effort="0" velocity="3.32"/>
     </joint>
     <joint name="${prefix}joint_3" type="revolute">
-      <origin xyz="0 0 ${link2_length}" rpy="0 ${M_PI/2} 0" />
+      <origin xyz="${link2_length} 0 0" rpy="0 0 0" />
       <parent link="${prefix}link_2"/>
       <child link="${prefix}link_3"/>
-      <axis xyz="0 1 0"/>
+      <axis xyz="0 0 1"/>
       <limit lower="-${M_PI/2}" upper="${M_PI/2}" effort="0" velocity="3.67"/>
     </joint>
     <joint name="${prefix}joint_4" type="revolute">
-      <origin xyz="0 0 ${link3_length}" rpy="0 0 0"/>
+      <origin xyz="${link3_length} 0 0" rpy="0 0 0"/>
       <parent link="${prefix}link_3"/>
       <child link="${prefix}link_4"/>
-      <axis xyz="0 -1 0"/>
+      <axis xyz="0 0 1"/>
       <limit lower="-${M_PI/2}" upper="${M_PI/2}" effort="0" velocity="6.98"/>
     </joint>
-    <joint name="${prefix}gripper" type="revolute">
-      <origin xyz="0 0 ${link4_length + gripper_offset}" rpy="0 0 0"/>
+    <joint name="${prefix}gripper" type="fixed">
+      <origin xyz="${link4_length + gripper_offset} 0 0" rpy="0 0 0"/>
       <parent link="${prefix}link_4"/>
       <child link="${prefix}gripper"/>
-      <axis xyz="-1 0 0"/>
+      <axis xyz="0 0 1"/>
       <limit lower="-${M_PI/2}" upper="${M_PI/2}" effort="0" velocity="6.98"/>
     </joint>
